File: Toasterboard.kicad_sch (KiCad schematic)
At the start: 0 parts

Commit message: feat: schematic progress! switches and leds done
Parts:
- added C1: 0.01uF, PCM_Capacitor_THT_US_AKL:C_Disc_D5.0mm_W2.5mm_P5.00mm, symbol PCM_Capacitor_US_AKL:C_Disc_D5.0mm_W2.5mm_P5.00mm
- added C2, C3: 100uF, PCM_Capacitor_THT_US_AKL:CP_Radial_D5.0mm_P2.00mm, symbol PCM_Capacitor_US_AKL:CP_Radial_D5.0mm_P2.00mm
- added J1: Power, symbol Connector_Generic:Conn_01x04
- added J2: LEDs, symbol Connector_Generic:Conn_01x04
- added J3: Switches, symbol Connector_Generic:Conn_01x04
- added LED1, LED2, LED3, LED4: Red, PCM_LED_THT_AKL:LED_D3.0mm, symbol PCM_LED_AKL:LED_3mm_Red
- added LED_CLK: Green, PCM_LED_THT_AKL:LED_D3.0mm, symbol PCM_LED_AKL:LED_3mm_Green
- added R_CLK, R_LED1, R_LED2, R_LED3, R_LED4: 1k, PCM_Resistor_THT_US_AKL:R_Axial_DIN0207_L6.3mm_D2.5mm_P5.08mm_Vertical, symbol PCM_Resistor_US_AKL:R_DIN0207_P5.08mm
- added SW1, SW2, SW3, SW4: SW_SPDT, symbol Switch:SW_SPDT
- added U1: LM341T-05_TO220, Package_TO_SOT_THT:TO-220-3_Vertical, symbol Regulator_Linear:LM341T-05_TO220
- added U2: NE555P, Package_DIP:DIP-8_W7.62mm, symbol Timer:NE555P
- added U3, U4: 74LS14, symbol 74xx:74LS14
Connections:
- new net: LED2.1 (K), R_LED2.1
- new net: J2.2 (Pin_2), LED2.2 (A)
- new net: C3.2, U2.2 (TRIG), U2.6 (THRES)
- new net: J3.1 (Pin_1), SW1.2 (B)
- new net: J3.2 (Pin_2), SW2.2 (B)
- new net: J3.3 (Pin_3), SW3.2 (B)
- new net: J3.4 (Pin_4), SW4.2 (B)
- new net: U3.2, U4.1
- new net: J2.1 (Pin_1), LED1.2 (A)
- new net: J2.3 (Pin_3), LED3.2 (A)
- new net: J2.4 (Pin_4), LED4.2 (A)
- new net: U2.3 (OUT), U3.1
- new net: LED1.1 (K), R_LED1.1
- new net: LED3.1 (K), R_LED3.1
- new net: LED_CLK.1 (K), R_CLK.1
- new net: LED4.1 (K), R_LED4.1
- new net +12V: J1.2 (Pin_2), U1.1 (VI)
- new net +5V: J1.1 (Pin_1), LED_CLK.2 (A), SW1.3 (C), SW2.3 (C), SW3.3 (C), SW4.3 (C), U1.3 (VO), U2.8 (VCC)
- new net Clk: J1.3 (Pin_3), R_CLK.2, U4.2
- new net GND: C3.1, J1.4 (Pin_4), R_LED1.2, R_LED2.2, R_LED3.2, R_LED4.2, SW1.1 (A), SW2.1 (A), SW3.1 (A), SW4.1 (A), U1.2 (GND), U2.1 (GND)
Other:
- company: (none) -> MatchaCircuits
- title: (none) -> Toasterboard
