File: shield/toastershield.kicad_pcb (KiCad board)
At the start: 2 copper layers, 68.6 x 53.3 mm, 31 parts, among them J1 Power, J2 Digital/PWM, J3 Analog, J4 Digital/PWM, SW1 SW_SPDT, SW2 SW_SPDT, SW3 SW_SPDT, SW4 SW_SPDT, U2 NE555P, U3 74HC14

Commit message: feat: i2c pullups on the shield
Parts:
- added R_PULLUP1: 5.1k, PCM_Resistor_THT_US_AKL:R_Axial_DIN0207_L6.3mm_D2.5mm_P2.54mm_Vertical, F.Cu at (112.0, 55.0)
- added R_PULLUP2: 5.1k, PCM_Resistor_THT_US_AKL:R_Axial_DIN0207_L6.3mm_D2.5mm_P2.54mm_Vertical, F.Cu at (117.5, 55.0)
- renumbered CLK to CLK_SOCK1
Connections:
- J2 pad 1: /SCL/A5/1 -> SCL/A5/1
- J2 pad 2: /SDA/A4/2 -> SDA/A4/2
Routing:
- net Net-(U2-THRES): track 53.4 -> 72.2 mm
- net +5V: track 198.1 -> 210.8 mm
- net SCL/A5/1: track 0.00 -> 7.63 mm
- net SDA/A4/2: track 0.00 -> 6.40 mm
Other:
- board text added: "12"
- board text added: "13"
- board text added: "2"
- board text added: "3.3V"
- board text added: "4"
- board text added: "5V"
- board text added: "7"
- board text added: "8"
- board text added: "A0"
- board text added: "A1"
- board text added: "A2"
- board text added: "A3"
- board text added: "A4"
- board text added: "A5"
- board text added: "AREF"
- board text added: "GND"
- board text added: "IOREF"
- board text added: "RESET"
- board text added: "RX<1"
- board text added: "SCL"
- board text added: "SDA"
- board text added: "TX>1"
- board text added: "Vin"
- board text added: "~10"
- board text added: "~11"
- board text added: "~3"
- board text added: "~5"
- board text added: "~6"
- board text added: "~9"

Commit message: feat: fix text and pins
Parts:
- added J5: PinHeader_2x03_P2.54mm_Vertical, Connector_PinHeader_2.54mm:PinHeader_2x03_P2.54mm_Vertical, B.Cu at (166.0, 69.5)
- added JB1: PinSocket_1x08_P2.54mm_Vertical, Connector_PinSocket_2.54mm:PinSocket_1x08_P2.54mm_Vertical, F.Cu at (128.0, 97.5)
- added JB2: PinSocket_1x10_P2.54mm_Vertical, Connector_PinSocket_2.54mm:PinSocket_1x10_P2.54mm_Vertical, F.Cu at (118.8, 49.2)
- added JB3: PinSocket_1x06_P2.54mm_Vertical, Connector_PinSocket_2.54mm:PinSocket_1x06_P2.54mm_Vertical, F.Cu at (150.8, 97.5)
- added JB4: PinSocket_1x08_P2.54mm_Vertical, Connector_PinSocket_2.54mm:PinSocket_1x08_P2.54mm_Vertical, F.Cu at (145.7, 49.2)
- added JB5: PinHeader_2x03_P2.54mm_Vertical, Connector_PinHeader_2.54mm:PinHeader_2x03_P2.54mm_Vertical, F.Cu at (163.5, 69.5)
- J1, J4: footprint Connector_PinSocket_2.54mm:PinSocket_1x08_P2.54mm_Vertical -> Connector_PinHeader_2.54mm:PinHeader_1x08_P2.54mm_Vertical
- J2: footprint Connector_PinSocket_2.54mm:PinSocket_1x10_P2.54mm_Vertical -> Connector_PinHeader_2.54mm:PinHeader_1x10_P2.54mm_Vertical
- J3: footprint Connector_PinSocket_2.54mm:PinSocket_1x06_P2.54mm_Vertical -> Connector_PinHeader_2.54mm:PinHeader_1x06_P2.54mm_Vertical
Other:
- board text added: "SHIELD"
- board text added: "Toasterboard"
- board text removed: "Toastershield"
