File: standalone/Toasterboard.kicad_pcb (KiCad board)
At the start: 2 copper layers, 64.5 x 46.5 mm, 33 parts, among them J1 Barrel Jack, J2 Power, J3 LEDs, J4 Switches, SW1 SW_SPDT, SW2 SW_SPDT, SW3 SW_SPDT, SW4 SW_SPDT

Commit message: feat: fix text and pins
Other:
- board text added: "5V"
- board text added: "CLK"
- board text added: "GND"
- board text added: "STANDALONE"
- board text added: "Vin"
Changed lines of the file:
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@@
 		(layer "Edge.Cuts")
+	)
+	(gr_text "STANDALONE"
+		(at 103.5 84.5 270)
+		(layer "F.SilkS")
+		(effects
+			(font
+				(size 0.5 0.5)
+				(thickness 0.125)
+			)
+			(justify right top)
+		)
+	)
+	(gr_text "Vin"
+		(at 126.5 68.5 90)
+		(layer "F.SilkS")
+		(effects
+			(font
+				(size 1 0.75)
+				(thickness 0.15)
+			)
+			(justify right bottom)
+		)
+	)
+	(gr_text "CLK"
+		(at 129 68.5 90)
+		(layer "F.SilkS")
+		(effects
+			(font
+				(size 1 0.75)
+				(thickness 0.15)
+			)
+			(justify right bottom)
+		)
+	)
+	(gr_text "GND"
+		(at 131.5 68.5 90)
+		(layer "F.SilkS")
+		(effects
+			(font
+				(size 1 0.75)
+				(thickness 0.15)
+			)
+			(justify right bottom)
+		)
 	)
 	(gr_text "R_USB"
@@
 		)
 	)
-	(gr_text "L4"
-		(at 142 71 90)
+	(gr_text "5V"
+		(at 124 68.5 90)
 		(layer "F.SilkS")
 		(effects
@@
 				(thickness 0.15)
 			)
-			(justify left bottom)
+			(justify right bottom)
 		)
 	)
-	(gr_text "L3"
-		(at 144.5 71 90)
+	(gr_text "L4"
+		(at 142 68.5 90)
 		(layer "F.SilkS")
 		(effects
@@
 				(thickness 0.15)
 			)
-			(justify left bottom)
+			(justify right bottom)
 		)
 	)
-	(gr_text "L2"
-		(at 147 71 90)
+	(gr_text "L3"
+		(at 144.5 68.5 90)
 		(layer "F.SilkS")
 		(effects
@@
 				(thickness 0.15)
 			)
-			(justify left bottom)
+			(justify right bottom)
 		)
 	)
-	(gr_text "L1"
-		(at 149.5 71 90)
+	(gr_text "L2"
+		(at 147 68.5 90)
 		(layer "F.SilkS")
 		(effects
@@
 				(thickness 0.15)
 			)
-			(justify left bottom)
+			(justify right bottom)
 		)
 	)
-	(gr_text "S4"
-		(at 154.5 71 90)
+	(gr_text "L1"
+		(at 149.5 68.5 90)
 		(layer "F.SilkS")
 		(effects
@@
 				(thickness 0.15)
 			)
-			(justify left bottom)
+			(justify right bottom)
 		)
 	)
-	(gr_text "S3"
-		(at 157 71 90)
+	(gr_text "S4"
+		(at 154.5 68.5 90)
 		(layer "F.SilkS")
 		(effects
@@
 				(thickness 0.15)
 			)
-			(justify left bottom)
+			(justify right bottom)
 		)
 	)
-	(gr_text "S2"
-		(at 159.5 71 90)
+	(gr_text "S3"
+		(at 157 68.5 90)
 		(layer "F.SilkS")
 		(effects
@@
 				(thickness 0.15)
 			)
-			(justify left bottom)
+			(justify right bottom)
 		)
 	)
-	(gr_text "S1"
-		(at 162 71 90)
+	(gr_text "S2"
+		(at 159.5 68.5 90)
 		(layer "F.SilkS")
 		(effects
@@
 				(thickness 0.15)
 			)
-			(justify left bottom)
+			(justify right bottom)
+		)
+	)
+	(gr_text "S1"
+		(at 162 68.5 90)
+		(layer "F.SilkS")
+		(effects
+			(font
+				(size 1 1)
+				(thickness 0.15)
+			)
+			(justify right bottom)
 		)
 	)
@@
 	)
 	(gr_text "Mk. I"
-		(at 104 85 270)
+		(at 104.000448 84.687219 270)
 		(layer "F.SilkS")
 		(effects
